File: sound-op-switch.brd (EAGLE design)
At the start: 50 x 50 mm, 35 parts, among them IC1 PIC12F1822, IC2 LM358D

Commit message: updates
Parts:
- moved PTC1 12.4 mm to (44.5, 31.0), turned to 90 degrees
- moved D2 2.54 mm to (44.5, 22.9)
- turned DET to 270 degrees
- turned PWR to 270 degrees
- turned R10 to 270 degrees
- turned R11 to 270 degrees
- turned R9 to 270 degrees
- turned TRG to 270 degrees
Routing:
- net N$19: track 3.57 -> 11.1 mm
- net GND: track 40.3 -> 47.7 mm, vias 5 -> 6
- net VCC: track 142.8 -> 149.8 mm, vias 0 -> 1
- net N$6: track 26.9 -> 22.1 mm
- net INPUT: track 60.9 -> 59.5 mm, vias 0 -> 1
- net N$4: track 2.89 -> 4.23 mm
- net N$17: track 2.89 -> 4.23 mm
- net N$16: track 2.89 -> 4.23 mm
- net N$7: track 32.1 -> 33.1 mm
- net N$3: track 23.6 -> 23.0 mm
Other:
- outline, holes or cut-outs redrawn
- board text added: "SOUND"
- board text added: "SWITCH"
- board text added: "hotchk155"
- board text added: "v1"
