File: sound-op-switch.sch (EAGLE design)
At the start: 35 parts, among them IC1 PIC12F1822, IC2 LM358D

Commit message: add device names and bom
Parts:
- C1: value (none) -> 4u7
- C3: value (none) -> 100u
- R1, R2, R3, R4, R5: value (none) -> 10k
- R10, R11, R9: value (none) -> 2k2
- R12: value 10k -> 1k
- R13: value (none) -> 1m
- R6: value (none) -> 470
- R7, R8: value 10k -> 2k2
- T1: value (none) -> MMBTA13
Changed lines of the file:
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@@
 <parts>
 <part name="MIC" library="pinhead" deviceset="PINHD-1X2" device=""/>
-<part name="R7" library="resistor" deviceset="R-EU_" device="R0805" value="10k"/>
-<part name="R12" library="rcl" deviceset="R-EU_" device="R0805" value="10k"/>
+<part name="R7" library="resistor" deviceset="R-EU_" device="R0805" value="2k2"/>
+<part name="R12" library="rcl" deviceset="R-EU_" device="R0805" value="1k"/>
 <part name="IC2" library="linear" deviceset="LM358" device="D" value="LM358D"/>
 <part name="GND1" library="supply1" deviceset="GND" device=""/>
@@
 <part name="GAIN" library="jasons_stuff" deviceset="ALPS_POT_SMALL" device=""/>
 <part name="EXT" library="jason_eagle6" deviceset="TRUCONNECTJACK" device=""/>
-<part name="R13" library="resistor" deviceset="R-EU_" device="R0805"/>
+<part name="R13" library="resistor" deviceset="R-EU_" device="R0805" value="1m"/>
 <part name="GND6" library="supply1" deviceset="GND" device=""/>
 <part name="ICSP" library="pinhead" deviceset="PINHD-1X6" device=""/>
 <part name="C2" library="resistor" deviceset="C-EU" device="C0805"/>
-<part name="R6" library="resistor" deviceset="R-EU_" device="R0805"/>
+<part name="R6" library="resistor" deviceset="R-EU_" device="R0805" value="470"/>
 <part name="GND7" library="supply1" deviceset="GND" device=""/>
 <part name="PWR" library="led" deviceset="LED" device="3MM"/>
-<part name="R11" library="resistor" deviceset="R-EU_" device="R0805"/>
+<part name="R11" library="resistor" deviceset="R-EU_" device="R0805" value="2k2"/>
 <part name="GND8" library="supply1" deviceset="GND" device=""/>
 <part name="OUT" library="jason_eagle6" deviceset="TRUCONNECTJACK" device=""/>
 <part name="RLY1" library="jason_eagle6" deviceset="9007-REED-RELAY" device=""/>
-<part name="R5" library="resistor" deviceset="R-EU_" device="R0805"/>
+<part name="R5" library="resistor" deviceset="R-EU_" device="R0805" value="10k"/>
 <part name="GND10" library="supply1" deviceset="GND" device=""/>
 <part name="MODE" library="jason_eagle6" deviceset="SP4T-SLIDE" device=""/>
-<part name="R1" library="resistor" deviceset="R-EU_" device="R0805"/>
-<part name="R4" library="resistor" deviceset="R-EU_" device="R0805"/>
-<part name="R3" library="resistor" deviceset="R-EU_" device="R0805"/>
+<part name="R1" library="resistor" deviceset="R-EU_" device="R0805" value="10k"/>
+<part name="R4" library="resistor" deviceset="R-EU_" device="R0805" value="10k"/>
+<part name="R3" library="resistor" deviceset="R-EU_" device="R0805" value="10k"/>
 <part name="GND5" library="supply1" deviceset="GND" device=""/>
 <part name="IC1" library="jasons_stuff" deviceset="PIC12F1822" device=""/>
-<part name="R8" library="resistor" deviceset="R-EU_" device="R0805" value="10k"/>
+<part name="R8" library="resistor" deviceset="R-EU_" device="R0805" value="2k2"/>
 <part name="GND9" library="supply1" deviceset="GND" device=""/>
-<part name="C3" library="rcl" deviceset="CPOL-EU" device="E2,5-6E"/>
+<part name="C3" library="rcl" deviceset="CPOL-EU" device="E2,5-6E" value="100u"/>
 <part name="THLD" library="jasons_stuff" deviceset="ALPS_POT_SMALL" device=""/>
 <part name="GND3" library="supply1" deviceset="GND" device=""/>
 <part name="DET" library="led" deviceset="LED" device="3MM"/>
-<part name="R9" library="resistor" deviceset="R-EU_" device="R0805"/>
+<part name="R9" library="resistor" deviceset="R-EU_" device="R0805" value="2k2"/>
 <part name="GND4" library="supply1" deviceset="GND" device=""/>
 <part name="TRG" library="led" deviceset="LED" device="3MM"/>
-<part name="R10" library="resistor" deviceset="R-EU_" device="R0805"/>
-<part name="R2" library="resistor" deviceset="R-EU_" device="R0805"/>
-<part name="C1" library="rcl" deviceset="CPOL-EU" device="E2,5-6E"/>
+<part name="R10" library="resistor" deviceset="R-EU_" device="R0805" value="2k2"/>
+<part name="R2" library="resistor" deviceset="R-EU_" device="R0805" value="10k"/>
+<part name="C1" library="rcl" deviceset="CPOL-EU" device="E2,5-6E" value="4u7"/>
 <part name="GND11" library="supply1" deviceset="GND" device=""/>
 <part name="ONOFF" library="pinhead" deviceset="PINHD-1X3" device=""/>
 <part name="BATT" library="pinhead" deviceset="PINHD-1X2" device=""/>
 <part name="GND12" library="supply1" deviceset="GND" device=""/>
-<part name="T1" library="transistor-neu-to92" deviceset="*-NPN-" device="SOT23-BEC" technology="MMBT3904LT1"/>
+<part name="T1" library="transistor-neu-to92" deviceset="*-NPN-" device="SOT23-BEC" technology="MMBT3904LT1" value="MMBTA13"/>
 <part name="D1" library="jasons_stuff" deviceset="0805DIODE" device=""/>
 <part name="PTC1" library="microbuilder" deviceset="PTC" device="1206"/>
@@
 <instance part="GND10" gate="1" x="53.34" y="-134.62"/>
 <instance part="MODE" gate="G$1" x="114.3" y="-17.78"/>
-<instance part="R1" gate="G$1" x="114.3" y="-38.1" rot="R90"/>
-<instance part="R4" gate="G$1" x="109.22" y="-38.1" rot="R90"/>
-<instance part="R3" gate="G$1" x="104.14" y="-38.1" rot="R90"/>
+<instance part="R1" gate="G$1" x="114.3" y="-38.1" smashed="yes" rot="R90">
+<attribute name="NAME" x="112.8014" y="-41.91" size="1.778" layer="95" rot="R90"/>
+<attribute name="VALUE" x="112.522" y="-36.83" size="1.778" layer="96" rot="R90"/>
+</instance>
+<instance part="R4" gate="G$1" x="109.22" y="-38.1" smashed="yes" rot="R90">
+<attribute name="NAME" x="107.7214" y="-41.91" size="1.778" layer="95" rot="R90"/>
+<attribute name="VALUE" x="107.442" y="-36.83" size="1.778" layer="96" rot="R90"/>
+</instance>
+<instance part="R3" gate="G$1" x="104.14" y="-38.1" smashed="yes" rot="R90">
+<attribute name="NAME" x="102.6414" y="-41.91" size="1.778" layer="95" rot="R90"/>
+<attribute name="VALUE" x="102.362" y="-36.83" size="1.778" layer="96" rot="R90"/>
+</instance>
 <instance part="GND5" gate="1" x="99.06" y="-50.8"/>
 <instance part="IC1" gate="G$1" x="5.08" y="-40.64"/>

Commit message: case proto
Parts:
- C3: value 100u -> 1u
Changed lines of the file:
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@@
 <part name="R8" library="resistor" deviceset="R-EU_" device="R0805" value="2k2"/>
 <part name="GND9" library="supply1" deviceset="GND" device=""/>
-<part name="C3" library="rcl" deviceset="CPOL-EU" device="E2,5-6E" value="100u"/>
+<part name="C3" library="rcl" deviceset="CPOL-EU" device="E2,5-6E" value="1u"/>
 <part name="THLD" library="jasons_stuff" deviceset="ALPS_POT_SMALL" device=""/>
 <part name="GND3" library="supply1" deviceset="GND" device=""/>

Commit message: pcb rev2
Parts:
- removed GAIN: ALPS_POT_SMALL, jasons_stuff:ALPS_POT_SMALL
- removed MODE: SP4T-SLIDE, jason_eagle6:SP4T-SLIDE
- removed T1: MMBTA13, transistor-neu-to92:MMBT3904LT1-NPN-SOT23-BEC
- added R14: 2k2, resistor:R-EU_R0805
- added SEL: SP4T-SLIDE, jason_eagle6:SP4T-SLIDE
- added TR1: MMBTA13, transistor-neu-to92:MMBT3904LT1-NPN-SOT23-BEC
- R10, R11, R8, R9: value 2k2 -> 10k
- R12: value 1k -> 470; device rcl:R-EU_R0805 -> resistor:R-EU_R0805
- R13: value 1m -> 2k2
- R2, R4: value 10k -> 2k2
- R3: value 10k -> 1m
- R5: value 10k -> 100k; device resistor:R-EU_R0805 -> rcl:R-EU_R0805
- R6: value 470 -> 1k; device resistor:R-EU_R0805 -> rcl:R-EU_R0805
Connections:
- net GND: now also R1.1, R13.1, R4.1, R7.1, R8.1, SEL.A, TR1.E; no longer MODE.A, R10.1, R11.1, R3.1, R5.1, R9.1, T1.E
- net INPUT: now also R3.2; no longer R13.2
- net N$1: now also R2.1; no longer R7.1
- net N$10: now also R1.2, R12.2, TR1.B; no longer R5.2, R6.2, T1.B
- net N$13: now also R3.1; no longer R13.1
- net N$14: now also R8.2, R9.1, SEL.B; no longer MODE.B, R3.2, R4.1
- net N$15: now also TR1.C; no longer T1.C
- net N$16: now also R4.2; no longer R11.2
- net N$17: now also R13.2; no longer R10.2
- net N$2: now also R6.2; no longer R12.2
- net N$3: now also R5.2, R6.1; no longer GAIN.A, R12.1
- net N$4: now also R7.2; no longer R9.2
- net N$5: now also R14.1; no longer R8.1
- net N$7: now also R5.1; no longer GAIN.B, GAIN.W
- net N$8: now also R10.1, R9.2, SEL.C; no longer MODE.C, R1.1, R4.2
- net N$9: now also R11.2; no longer R2.2
- net OUTPUT: now also R12.1; no longer R6.1
- net VCC: now also R10.2, R14.2, R2.2; no longer R1.2, R7.2, R8.2
- net VSEL: now also R11.1, SEL.COM; no longer MODE.COM, R2.1
Other:
- note added: "INPUT & PRE-AMP"
- note added: "J HOTCHKISS"
- note added: "MODE SELECT"
- note added: "OUTPUT SWITCH"
- note added: "POWER INPUT & POLARITY PROTECY"
- note added: "PROCESSOR"
- note added: "SHOUTBOX V2"
- moved on the sheet: BATT, C1, C3, D2, DET, EXT, IC2A, IC2B, MIC, ONOFF, OUT, PTC1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
