File: hardware/sound-op-switch.brd (EAGLE design)
At the start: 50 x 50 mm, 35 parts, among them IC1 PIC12F1822, IC2 LM358D

Commit message: REV3
fix mic position
Parts:
- R13, R4, R7: value 2k2 -> 1k
- moved MIC 4.39 mm to (3.56, 25.0)
Routing:
- net INPUT: track 73.5 -> 68.4 mm
- net N$1: track 35.0 -> 38.9 mm
Other:
- board text added: "rev3"
- board text added: "sound operated switch"
- board text removed: "SHOUTBOX"
- board text removed: "rev2"
Changed lines of the file:
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@@
 <wire x1="0" y1="47.371" x2="0" y2="47.498" width="0.254" layer="20"/>
 <wire x1="0" y1="47.498" x2="2.54" y2="49.9872" width="0.254" layer="20" curve="-90"/>
-<text x="18.034" y="4.3434" size="1.778" layer="25" font="vector" rot="R180">SHOUTBOX</text>
-<text x="41.6306" y="2.159" size="1.27" layer="25" font="vector" rot="R180">hotchk155</text>
+<text x="5.3594" y="2.5908" size="1.27" layer="25" font="vector">hotchk155</text>
 <circle x="45.6438" y="21.717" radius="0.851940625" width="0.254" layer="21"/>
 <wire x1="45.2628" y1="21.6916" x2="46.0248" y2="21.6916" width="0.254" layer="21"/>
-<text x="17.907" y="4.2672" size="1.778" layer="25" font="vector" rot="R180">SHOUTBOX</text>
-<text x="18.2118" y="2.4384" size="1.27" layer="25" font="vector" rot="R180">rev2</text>
+<text x="28.3464" y="1.9304" size="1.27" layer="25" font="vector" rot="R180">sound operated switch</text>
+<text x="36.9316" y="2.0066" size="1.27" layer="25" font="vector" rot="R180">rev3</text>
 </plain>
 <attributes>
@@
 </class>
 </classes>
-<designrules name="ITEADstudio_DRC">
-<description language="de">&lt;b&gt;EAGLE Design Rules&lt;/b&gt;
+<designrules name="hackvana">
+<description language="de">&lt;b&gt;EAGLE Design Rules für Hackvana&lt;/b&gt;
 &lt;p&gt;
 Die Standard-Design-Rules sind so gewählt, dass sie für
@@
 Einstellungen hier und speichern die Design Rules unter
 einem neuen Namen ab.</description>
-<description language="en">&lt;b&gt;EAGLE Design Rules&lt;/b&gt;
+<description language="en">&lt;b&gt;EAGLE Design Rules for Hackvana&lt;/b&gt;
 &lt;p&gt;
 The default Design Rules have been set to cover
@@
 necessary adjustments and save your customized
 design rules under a new name.</description>
-<description language="zh">&lt;b&gt;Seeed Studio EAGLE Design Rules&lt;/b&gt;
+<description language="zh">&lt;b&gt;EAGLE Design Rules for Hackvana&lt;/b&gt;
 </description>
 <param name="layerSetup" value="(1*16)"/>
@@
 <param name="mdViaViaSameLayer" value="8mil"/>
 <param name="mnLayersViaInSmd" value="2"/>
-<param name="mdCopperDimension" value="10mil"/>
-<param name="mdDrill" value="10mil"/>
+<param name="mdCopperDimension" value="6mil"/>
+<param name="mdDrill" value="6mil"/>
 <param name="mdSmdStop" value="0mil"/>
 <param name="msWidth" value="6mil"/>
-<param name="msDrill" value="12mil"/>
-<param name="msMicroVia" value="12mil"/>
+<param name="msDrill" value="0.3mm"/>
+<param name="msMicroVia" value="0.25mm"/>
 <param name="msBlindViaRatio" value="0.5"/>
 <param name="rvPadTop" value="0.25"/>
@@
 </autorouter>
 <elements>
-<element name="MIC" library="pinhead" package="1X02" value="" x="7.9502" y="24.9936" smashed="yes" rot="R90">
-<attribute name="NAME" x="5.7658" y="25.6794" size="1.27" layer="25" ratio="10" rot="R180"/>
-<attribute name="VALUE" x="11.1252" y="22.4536" size="1.27" layer="27" rot="R90"/>
+<element name="MIC" library="pinhead" package="1X02" value="" x="3.556" y="24.9936" smashed="yes" rot="R90">
+<attribute name="NAME" x="8.9916" y="25.6794" size="1.27" layer="25" ratio="10" rot="R180"/>
+<attribute name="VALUE" x="6.731" y="22.4536" size="1.27" layer="27" rot="R90"/>
 </element>
 <element name="R2" library="resistor" package="R0805" value="2k2" x="15.24" y="36.7284" smashed="yes">
@@
 <attribute name="VALUE" x="13.589" y="30.7086" size="1.27" layer="27" ratio="10" rot="R270"/>
 </element>
-<element name="R4" library="resistor" package="R0805" value="2k2" x="15.24" y="28.956" smashed="yes" rot="R180">
+<element name="R4" library="resistor" package="R0805" value="1k" x="15.24" y="28.956" smashed="yes" rot="R180">
 <attribute name="NAME" x="10.6172" y="28.3464" size="1.27" layer="25"/>
 </element>
@@
 <attribute name="VALUE" x="13.589" y="23.0886" size="1.27" layer="27" ratio="10" rot="R270"/>
 </element>
-<element name="R7" library="resistor" package="R0805" value="2k2" x="15.24" y="20.9042" smashed="yes" rot="R180">
+<element name="R7" library="resistor" package="R0805" value="1k" x="15.24" y="20.9042" smashed="yes" rot="R180">
 <attribute name="NAME" x="12.8778" y="21.3868" size="1.27" layer="25" rot="R180"/>
 </element>
@@
 <attribute name="VALUE" x="13.589" y="15.4686" size="1.27" layer="27" ratio="10" rot="R270"/>
 </element>
-<element name="R13" library="resistor" package="R0805" value="2k2" x="15.24" y="12.4968" smashed="yes" rot="R180">
+<element name="R13" library="resistor" package="R0805" value="1k" x="15.24" y="12.4968" smashed="yes" rot="R180">
 <attribute name="NAME" x="13.6652" y="13.716" size="1.27" layer="25"/>
 </element>
@@
 <contactref element="R2" pad="1"/>
 <contactref element="EXT" pad="TIP_NC"/>
-<wire x1="7.9502" y1="26.2636" x2="9.7536" y2="26.2636" width="0.4064" layer="1"/>
+<wire x1="3.556" y1="26.2636" x2="6.35" y2="26.2636" width="0.4064" layer="1"/>
+<wire x1="6.35" y1="26.2636" x2="9.7536" y2="26.2636" width="0.4064" layer="1"/>
 <wire x1="9.7536" y1="26.2636" x2="11.43" y2="27.94" width="0.4064" layer="1"/>
 <wire x1="11.43" y1="27.94" x2="11.43" y2="33.7684" width="0.4064" layer="1"/>
 <wire x1="11.43" y1="33.7684" x2="14.39" y2="36.7284" width="0.4064" layer="1"/>
-<wire x1="7.9502" y1="26.2636" x2="5.9436" y2="26.2636" width="0.4064" layer="1"/>
-<wire x1="5.9436" y1="26.2636" x2="5.08" y2="25.4" width="0.4064" layer="1"/>
-<wire x1="5.08" y1="25.4" x2="5.08" y2="20.32" width="0.4064" layer="1"/>
-<wire x1="5.08" y1="20.32" x2="6.35" y2="19.05" width="0.4064" layer="1"/>
-<wire x1="6.35" y1="19.05" x2="6.35" y2="11.938" width="0.4064" layer="1"/>
+<wire x1="3.556" y1="26.2636" x2="5.9436" y2="26.2636" width="0.4064" layer="1"/>
+<wire x1="6.35" y1="26.2636" x2="6.35" y2="11.938" width="0.4064" layer="1"/>
 <wire x1="6.35" y1="11.938" x2="8.89" y2="9.398" width="0.4064" layer="1"/>
 </signal>
@@
 <wire x1="24.98" y1="32.5374" x2="24.9546" y2="32.5628" width="0.4064" layer="1"/>
 <wire x1="18.7452" y1="8.89" x2="13.7414" y2="3.8862" width="0.4064" layer="16"/>
-<wire x1="13.7414" y1="3.8862" x2="6.7564" y2="3.8862" width="0.4064" layer="16"/>
-<wire x1="6.7564" y1="3.8862" x2="6.096" y2="4.5466" width="0.4064" layer="16"/>
-<wire x1="6.096" y1="4.5466" x2="6.096" y2="19.304" width="0.4064" layer="16"/>
-<wire x1="6.096" y1="19.304" x2="5.08" y2="20.32" width="0.4064" layer="16"/>
-<wire x1="5.08" y1="20.32" x2="5.08" y2="26.67" width="0.4064" layer="16"/>
-<wire x1="5.08" y1="26.67" x2="6.35" y2="27.94" width="0.4064" layer="16"/>
-<wire x1="6.35" y1="27.94" x2="13.208" y2="27.94" width="0.4064" layer="16"/>
-<wire x1="13.208" y1="27.94" x2="15.24" y2="26.2636" width="0.4064" layer="16"/>
 <wire x1="15.24" y1="26.2636" x2="26.2636" y2="26.2636" width="0.4064" layer="16"/>
 <wire x1="26.2636" y1="26.2636" x2="27.94" y2="27.94" width="0.4064" layer="16"/>
 <wire x1="18.7452" y1="8.89" x2="20.32" y2="8.89" width="0.4064" layer="16"/>
+<wire x1="13.7414" y1="3.8862" x2="7.5438" y2="3.8862" width="0.4064" layer="16"/>
+<wire x1="7.5438" y1="3.8862" x2="6.35" y2="5.08" width="0.4064" layer="16"/>
+<wire x1="6.35" y1="5.08" x2="6.35" y2="24.13" width="0.4064" layer="16"/>
+<wire x1="15.24" y1="26.2636" x2="8.4836" y2="26.2636" width="0.4064" layer="16"/>
+<wire x1="8.4836" y1="26.2636" x2="6.35" y2="24.13" width="0.4064" layer="16"/>
 </signal>
 <signal name="N$4">
