File: hardware/sound-op-switch.sch (EAGLE design)
At the start: 35 parts, among them IC1 PIC12F1822, IC2 LM358D

Commit message: REV3
fix mic position
Parts:
- R13, R4, R7: value 2k2 -> 1k
Changed lines of the file:
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@@
 <part name="GND7" library="supply1" deviceset="GND" device=""/>
 <part name="PWR" library="led" deviceset="LED" device="3MM"/>
-<part name="R4" library="resistor" deviceset="R-EU_" device="R0805" value="2k2"/>
+<part name="R4" library="resistor" deviceset="R-EU_" device="R0805" value="1k"/>
 <part name="GND8" library="supply1" deviceset="GND" device=""/>
 <part name="OUT" library="jason_eagle6" deviceset="TRUCONNECTJACK" device=""/>
@@
 <part name="GND3" library="supply1" deviceset="GND" device=""/>
 <part name="DET" library="led" deviceset="LED" device="3MM"/>
-<part name="R7" library="resistor" deviceset="R-EU_" device="R0805" value="2k2"/>
+<part name="R7" library="resistor" deviceset="R-EU_" device="R0805" value="1k"/>
 <part name="GND4" library="supply1" deviceset="GND" device=""/>
 <part name="TRG" library="led" deviceset="LED" device="3MM"/>
-<part name="R13" library="resistor" deviceset="R-EU_" device="R0805" value="2k2"/>
+<part name="R13" library="resistor" deviceset="R-EU_" device="R0805" value="1k"/>
 <part name="R11" library="resistor" deviceset="R-EU_" device="R0805" value="10k"/>
 <part name="C1" library="rcl" deviceset="CPOL-EU" device="E2,5-6E" value="4u7"/>
